Commit message: LEFT & RIGHT Link and Joint

File: my_robot/urdf/my_robot.xacro (robot description, xacro)
@@ -55,5 +55,5 @@
   </link>
   <!--MY LEFT Link and JOINT-->
-  <link name='SIDE_wheel'>
+  <link name='LEFT_wheel'>
     <pose>0 0 0.1 0 0 0</pose>
     <inertial>
@@ -67,10 +67,10 @@
     </inertial>
     <collision name='collision'>
-      <origin xyz="0 0 0" rpy=" 0 0 0"/>
+      <origin xyz="0 0 0" rpy=" 0 0.7505 0.7505"/>
       <geometry>
         <box size=".4 .2 .1"/>
       </geometry>
     </collision>
-    <visual name='SIDE_wheel_visual'>
+    <visual name='LEFT_wheel_visual'>
       <origin xyz="0.0 0 0" rpy=" 0 1.5707 1.5707"/>
       <geometry>
@@ -79,7 +79,7 @@
     </visual>
   </link>
-  <joint type="continuous" name="left_wheel_hinge">
+  <joint type="continuous" name="LEFT_wheel_hinge">
     <origin xyz="0 0.15 0" rpy="0 0 0"/>
-    <child link="left_wheel"/>
+    <child link="LEFT_wheel"/>
     <parent link="chassis"/>
     <axis xyz="0 1 0" rpy="0 0 0"/>
@@ -89,5 +89,5 @@
   <!--MY LEFT Link and JOINT-->
   <!--MY RIGHT Link and JOINT-->
-  <link name='SIDE_wheel'>
+  <link name='RIGHT_wheel'>
     <pose>0 0 0.1 0 0 0</pose>
     <inertial>
@@ -101,10 +101,10 @@
     </inertial>
     <collision name='collision'>
-      <origin xyz="0 0 0" rpy=" 0 0 0"/>
+      <origin xyz="0 0 0" rpy=" 0 0.7505 0.7505"/>
       <geometry>
         <box size=".4 .2 .1"/>
       </geometry>
     </collision>
-    <visual name='SIDE_wheel_visual'>
+    <visual name='RIGHT_wheel_visual'>
       <origin xyz="0.0 0 0" rpy=" 0 1.5707 1.5707"/>
       <geometry>
@@ -113,7 +113,7 @@
     </visual>
   </link>
-  <joint type="continuous" name="left_wheel_hinge">
+  <joint type="continuous" name="RIGHT_wheel_hinge">
     <origin xyz="0 0.15 0" rpy="0 0 0"/>
-    <child link="right_wheel"/>
+    <child link="RIGHT_wheel"/>
     <parent link="chassis"/>
     <axis xyz="0 1 0" rpy="0 0 0"/>

Commit message: Add files via upload

File: my_robot/urdf/my_robot.xacro (robot description, xacro)
@@ -80,5 +80,5 @@
   </link>
   <joint type="continuous" name="LEFT_wheel_hinge">
-    <origin xyz="0 0.15 0" rpy="0 0 0"/>
+    <origin xyz="0 0.125 0" rpy="0 0 0"/>
     <child link="LEFT_wheel"/>
     <parent link="chassis"/>
@@ -101,5 +101,5 @@
     </inertial>
     <collision name='collision'>
-      <origin xyz="0 0 0" rpy=" 0 0.7505 0.7505"/>
+      <origin xyz="0 0 0" rpy=" 0 2.3562 2.3562"/>
       <geometry>
         <box size=".4 .2 .1"/>
@@ -114,5 +114,5 @@
   </link>
   <joint type="continuous" name="RIGHT_wheel_hinge">
-    <origin xyz="0 0.15 0" rpy="0 0 0"/>
+    <origin xyz="0 -0.125 0" rpy="0 0 0"/>
     <child link="RIGHT_wheel"/>
     <parent link="chassis"/>
@@ -122,3 +122,71 @@
   </joint>
   <!--MY RIGHT Link and JOINT-->
+  <!--MY CAMERA Link and JOINT-->
+  <link name='camera'>
+    <pose>0 0 0 0 0 0</pose>
+    <inertial>
+      <mass value="0.1"/>
+      <origin xyz="0.05 0.05 0.05" rpy=" 0 0 0"/>
+      <inertia
+          ixx="1e-6" ixy="0" ixz="0"
+          iyy="1e-6" iyz="0"
+          izz="1e-6"
+      />
+    </inertial>
+    <collision name='camera_collision'>
+      <origin xyz="0 0 0" rpy=" 0 0 0"/>
+      <geometry>
+        <box size="0.1 0.1 0.1"/>
+      </geometry>
+    </collision>
+    <visual name='camera_visual'>
+      <origin xyz="0 0 0" rpy=" 0 0 0"/>
+      <geometry>
+        <box size="0.05 0.05 0.05"/>
+      </geometry>
+    </visual>
+  </link>
+  <joint type="fixed" name="camera_joint">
+    <origin xyz="0.2 0 0" rpy="0 0 0"/>
+    <child link="camera"/>
+    <parent link="chassis"/>
+    <axis xyz="0 1 0" rpy="0 0 0"/>
+    <limit effort="10000" velocity="1000"/>
+    <dynamics damping="1.0" friction="1.0"/>
+  </joint>
+  <!--MY CAMERA Link and JOINT-->
+  <!--MY HOKUYO Link and JOINT-->
+  <link name='hokuyo'>
+    <pose>0 0 0 0 0 0</pose>
+    <inertial>
+      <mass value="1e-5"/>
+      <origin xyz="0 0 0" rpy=" 0 0 0"/>
+      <inertia
+          ixx="1e-6" ixy="0" ixz="0"
+          iyy="1e-6" iyz="0"
+          izz="1e-6"
+      />
+    </inertial>
+    <collision name='hokuyo_collision'>
+      <origin xyz="0 0 0" rpy=" 0 0 0"/>
+      <geometry>
+        <box size="0.1 0.1 0.1"/>
+      </geometry>
+    </collision>
+    <visual name='hokuyo_visual'>
+      <origin xyz="0 0 0" rpy=" 0 0 0"/>
+      <geometry>
+        <mesh filename=“package://home/robond/catkin_ws/src/my_robot/meshes/hokuyo.dae”/>
+      </geometry>
+    </visual>
+  </link>
+  <joint type="fixed" name="hokuyo_joint">
+    <origin xyz="0.15 0 0.1" rpy="0 0 0"/>
+    <child link="hokuyo"/>
+    <parent link="chassis"/>
+    <axis xyz="0 1 0" rpy="0 0 0"/>
+    <limit effort="10000" velocity="1000"/>
+    <dynamics damping="1.0" friction="1.0"/>
+  </joint>
+  <!--MY HOKUYO Link and JOINT-->
 </robot>

Commit message: Add files via upload

File: my_robot/urdf/my_robot.xacro (robot description, xacro)
@@ -1,3 +1,6 @@
 <robot name="my_robot" xmlns:xacro="http://www.ros.org/wiki/xacro">
+  <!--MY GAZEBO PLUGINS-->
+  <xacro:include filename="$(find my_robot)/urdf/my_robot.gazebo" />
+  <!--MY GAZEBO PLUGINS-->
   <link name="robot_footprint"></link>
   <joint name="robot_footprint_joint" type="fixed">
@@ -177,10 +180,10 @@
       <origin xyz="0 0 0" rpy=" 0 0 0"/>
       <geometry>
-        <mesh filename=“package://home/robond/catkin_ws/src/my_robot/meshes/hokuyo.dae”/>
+        <mesh filename="package://my_robot/meshes/hokuyo.dae"/>
       </geometry>
     </visual>
   </link>
   <joint type="fixed" name="hokuyo_joint">
-    <origin xyz="0.15 0 0.1" rpy="0 0 0"/>
+    <origin xyz="0.15 0 0.08" rpy="0 0 0"/>
     <child link="hokuyo"/>
     <parent link="chassis"/>

Commit message: Add files via upload

File: my_robot/urdf/my_robot.xacro (robot description, xacro)
@@ -82,5 +82,5 @@
     </visual>
   </link>
-  <joint type="continuous" name="LEFT_wheel_hinge">
+  <joint type="continuous" name="left_wheel_hinge">
     <origin xyz="0 0.125 0" rpy="0 0 0"/>
     <child link="LEFT_wheel"/>
@@ -116,5 +116,5 @@
     </visual>
   </link>
-  <joint type="continuous" name="RIGHT_wheel_hinge">
+  <joint type="continuous" name="right_wheel_hinge">
     <origin xyz="0 -0.125 0" rpy="0 0 0"/>
     <child link="RIGHT_wheel"/>

Commit message: Add files via upload

File: my_robot/urdf/my_robot.xacro (robot description, xacro)
@@ -69,8 +69,8 @@
       />
     </inertial>
-    <collision name='collision'>
+    <collision name='LEFT_wheel_collision'>
       <origin xyz="0 0 0" rpy=" 0 0.7505 0.7505"/>
       <geometry>
-        <box size=".4 .2 .1"/>
+        <cylinder length="0.05" radius="0.1"/>
       </geometry>
     </collision>
@@ -103,8 +103,8 @@
       />
     </inertial>
-    <collision name='collision'>
+    <collision name='RIGHT_wheel_collision'>
       <origin xyz="0 0 0" rpy=" 0 2.3562 2.3562"/>
       <geometry>
-        <box size=".4 .2 .1"/>
+        <cylinder length="0.05" radius="0.1"/>
       </geometry>
     </collision>
